Commit message: feat: generate mapping from slam

File: p3at_description/urdf/hokuyo_utm30lx.urdf.xacro (robot description, xacro)
@@ -8,4 +8,10 @@
         <child link="${name}_frame"/>
       </joint>
+      <!-- <joint name="${name}_joint" type="revolute">
+        <xacro:insert_block name="origin" />
+        <parent link="${parent}" />
+        <child link="${name}_frame" />
+        <limit lower="0" upper="0" effort="0" velocity="0" />
+      </joint> -->
       <link name="${name}_frame">
         <inertial>
@@ -56,7 +62,7 @@
           </plugin>
         </sensor>
-        <plugin name="joint_state_publisher" filename="libgazebo_ros_joint_state_publisher.so" >
-            <jointName>hokuyo_joint</jointName>
-        </plugin>
+        <!-- <plugin name="joint_state_publisher" filename="libgazebo_ros_joint_state_publisher.so" >
+            <jointName>${name}_joint</jointName>
+        </plugin> -->
       </gazebo>
     </xacro:macro>

Commit message: fix: update original pioneer urdf xacros

File: p3at_description/urdf/hokuyo_utm30lx.urdf.xacro (robot description, xacro)
@@ -8,10 +8,4 @@
         <child link="${name}_frame"/>
       </joint>
-      <!-- <joint name="${name}_joint" type="revolute">
-        <xacro:insert_block name="origin" />
-        <parent link="${parent}" />
-        <child link="${name}_frame" />
-        <limit lower="0" upper="0" effort="0" velocity="0" />
-      </joint> -->
       <link name="${name}_frame">
         <inertial>
@@ -34,5 +28,5 @@
       </link>
       <gazebo reference="${name}_frame">
-        <sensor type="ray" name="${name}">
+        <sensor type="ray" name="${name}_sensor">
           <always_on>true</always_on>
           <update_rate>${update_rate}</update_rate>
@@ -62,7 +56,4 @@
           </plugin>
         </sensor>
-        <!-- <plugin name="joint_state_publisher" filename="libgazebo_ros_joint_state_publisher.so" >
-            <jointName>${name}_joint</jointName>
-        </plugin> -->
       </gazebo>
     </xacro:macro>

File: p3at_description/urdf/pioneer3at.urdf.xacro (robot description, xacro)
@@ -8,5 +8,6 @@
   <xacro:include filename="$(find p3at_description)/urdf/pioneer3at_body.xacro"/>
   <xacro:include filename="$(find p3at_description)/urdf/hokuyo_utm30lx.urdf.xacro"/>
-  <xacro:hokuyo_utm30lx name="hokuyo" parent="base_link" ros_topic="hokuyo" update_rate="30" ray_count="1040" min_angle="180" max_angle="-180" >
+  <xacro:pioneer3at_body/>
+  <xacro:hokuyo_utm30lx name="hokuyo" parent="base_link" ros_topic="hokuyo" update_rate="10" ray_count="1040" min_angle="180" max_angle="-180" >
     <origin xyz="0.13 0 0.32" rpy="0 0 0"/>
   </xacro:hokuyo_utm30lx>

File: p3at_description/urdf/pioneer3at_body.xacro (robot description, xacro)
@@ -1,163 +1,180 @@
 <?xml version="1.0"?>
-<robot xmlns:sensor="http://playerstage.sourceforge.net/gazebo/xmlschema/#sensor"
-  xmlns:controller="http://playerstage.sourceforge.net/gazebo/xmlschema/#controller"
-  xmlns:interface="http://playerstage.sourceforge.net/gazebo/xmlschema/#interface"
-  xmlns:xacro="http://ros.org/wiki/xacro"
-  >
-  <!-- Chassis -->
-  <link name="base_link">
-    <inertial>
-      <mass value="14.0"/>
-      <origin xyz="0 0 0.177"/>
-      <inertia ixx="0.14711667" ixy="0.0" ixz="0.0"
-        iyy="0.334951167" iyz="0.0"
-        izz="0.3978345"/>
-    </inertial>
-    <visual name="base_visual">
-      <origin xyz="0 0 0.18" rpy="0 0 0"/>
-      <geometry name="pioneer_geom">
-        <mesh filename="package://p3at_description/meshes/p3at_meshes/chassis.dae"/>
-      </geometry>
-    </visual>
-    <collision>
-      <origin xyz="0 0 0.18" rpy="0 0 0"/>
-      <geometry>
-        <box size="0.501 0.3 0.19"/>
-      </geometry>
-    </collision>
-  </link>
-  <link name="p3at_front_left_wheel">
-    <inertial>
-      <mass value="1.5"/>
-      <origin xyz="0 0 0"/>
-      <inertia ixx="0.005240625" ixy="0" ixz="0"
-        iyy="0.005240625" iyz="0" izz="0.009075"/>
-    </inertial>
-    <visual name="visual">
-      <origin xyz="0 0 0" rpy="0 0 0"/>
-      <geometry name="geom">
-        <mesh filename="package://p3at_description/meshes/p3at_meshes/wheel.dae"/>
-      </geometry>
-    </visual>
-    <collision>
-      <origin xyz="0 0 0" rpy="0 0 0"/>
-      <geometry>
-        <cylinder radius="0.110" length="0.075"/>
-      </geometry>
-    </collision>
-  </link>
-  <joint name="p3at_front_left_wheel_joint" type="continuous">
-    <axis xyz="0 0 -1"/>
-    <limit effort="100" velocity="100" />
-    <joint_properties damping="0.7"/>
-    <origin xyz="0.125 0.2010 0.11" rpy="1.5707 0 0"/>
-    <parent link="base_link"/>
-    <child link="p3at_front_left_wheel"/>
-  </joint>
-  <link name="p3at_front_right_wheel">
-    <inertial>
-      <mass value="1.5"/>
-      <origin xyz="0 0 0"/>
-      <inertia ixx="0.005240625" ixy="0" ixz="0"
-        iyy="0.005240625" iyz="0" izz="0.009075"/>
-    </inertial>
-    <visual name="visual">
-      <origin xyz="0 0 0" rpy="0 0 0"/>
-      <geometry name="geom">
-        <mesh filename="package://p3at_description/meshes/p3at_meshes/wheel.dae"/>
-      </geometry>
-    </visual>
-    <collision>
-      <origin xyz="0 0 0" rpy="0 0 0"/>
-      <geometry>
-        <cylinder radius="0.110" length="0.075"/>
-      </geometry>
-    </collision>
-  </link>
-  <joint name="p3at_front_right_wheel_joint" type="continuous">
-    <axis xyz="0 0 -1"/>
-    <limit effort="100" velocity="100" />
-    <joint_properties damping="0.7"/>
-    <origin xyz="0.125 -0.2010 0.11" rpy="1.5707 0 0"/>
-    <parent link="base_link"/>
-    <child link="p3at_front_right_wheel"/>
-  </joint>
-  <link name="p3at_rear_left_wheel">
-    <inertial>
-      <mass value="1.5"/>
-      <origin xyz="0 0 0"/>
-      <inertia ixx="0.005240625" ixy="0" ixz="0"
-        iyy="0.005240625" iyz="0" izz="0.009075"/>
-    </inertial>
-    <visual name="visual">
-      <origin xyz="0 0 0" rpy="0 0 0"/>
-      <geometry name="geom">
-        <mesh filename="package://p3at_description/meshes/p3at_meshes/wheel.dae"/>
-      </geometry>
-    </visual>
-    <collision>
-      <origin xyz="0 0 0" rpy="0 0 0"/>
-      <geometry>
-        <cylinder radius="0.110" length="0.075"/>
-      </geometry>
-    </collision>
-  </link>
-  <joint name="p3at_rear_left_wheel_joint" type="continuous">
-    <axis xyz="0 0 -1"/>
-    <limit effort="100" velocity="100" />
-    <joint_properties damping="0.7"/>
-    <origin xyz="-0.125 0.2010 0.11" rpy="1.5707 0 0"/>
-    <parent link="base_link"/>
-    <child link="p3at_rear_left_wheel"/>
-  </joint>
-  <link name="p3at_rear_right_wheel">
-    <inertial>
-      <mass value="1.5"/>
-      <origin xyz="0 0 0"/>
-      <inertia ixx="0.005240625" ixy="0" ixz="0"
-        iyy="0.005240625" iyz="0" izz="0.009075"/>
-    </inertial>
-    <visual name="visual">
-      <origin xyz="0 0 0" rpy="0 0 0"/>
-      <geometry name="geom">
-        <mesh filename="package://p3at_description/meshes/p3at_meshes/wheel.dae"/>
-      </geometry>
-    </visual>
-    <collision>
-      <origin xyz="0 0 0" rpy="0 0 0"/>
-      <geometry>
-        <cylinder radius="0.110" length="0.075"/>
-      </geometry>
-    </collision>
-  </link>
-  <joint name="p3at_rear_right_wheel_joint" type="continuous">
-    <axis xyz="0 0 -1"/>
-    <limit effort="100" velocity="100" />
-    <joint_properties damping="0.7"/>
-    <origin xyz="-0.125 -0.2010 0.11" rpy="1.5707 0 0"/>
-    <parent link="base_link"/>
-    <child link="p3at_rear_right_wheel"/>
-  </joint>
-  <gazebo>
-    <plugin name="skid_steer_drive_controller" filename="libgazebo_ros_skid_steer_drive.so">
-      <updateRate>100.0</updateRate>
-      <robotNamespace>$(arg robot_name)</robotNamespace>
-      <leftFrontJoint>p3at_front_left_wheel_joint</leftFrontJoint>
-      <rightFrontJoint>p3at_front_right_wheel_joint</rightFrontJoint>
-      <leftRearJoint>p3at_rear_left_wheel_joint</leftRearJoint>
-      <rightRearJoint>p3at_rear_right_wheel_joint</rightRearJoint>
-      <wheelSeparation>0.4</wheelSeparation>
-      <wheelDiameter>0.215</wheelDiameter>
-      <robotBaseFrame>base_link</robotBaseFrame>
-      <torque>200</torque>
-      <commandTopic>cmd_vel</commandTopic>
-      <odometryTopic>odom</odometryTopic>
-      <odometryFrame>odom</odometryFrame>
-      <broadcastTF>true</broadcastTF>
-      <publishWheelJointState>true</publishWheelJointState>
-    </plugin>
-    <!-- <plugin name="joint_state_publisher" filename="libgazebo_ros_joint_state_publisher.so" >
-      <jointName>p3at_front_left_wheel_joint, p3at_front_right_wheel_joint, p3at_rear_left_wheel_joint, p3at_rear_right_wheel_joint</jointName>
-    </plugin> -->
-  </gazebo>
+<robot xmlns:xacro="http://ros.org/wiki/xacro">
+  <xacro:macro name="pioneer3at_body">
+    <link name="base_footprint">
+      <visual>
+        <origin rpy="0 0 0" xyz="0 0 0"/>
+        <geometry>
+          <box size="0.001 0.001 0.001"/>
+        </geometry>
+      </visual>
+    </link>
+    <joint name="base_footprint_joint" type="fixed">
+      <origin rpy="0 0 0" xyz="0 0 0.127"/>
+      <!-- ${wheel_radius} property must be defined inside wheel description -->
+      <parent link="base_footprint"/>
+      <child link="base_link"/>
+    </joint>
+    <!-- Chassis -->
+    <link name="base_link">
+      <inertial>
+        <mass value="14.0"/>
+        <origin xyz="0 0 0.177"/>
+        <inertia ixx="0.14711667" ixy="0.0" ixz="0.0"
+          iyy="0.334951167" iyz="0.0"
+          izz="0.3978345"/>
+      </inertial>
+      <visual name="base_visual">
+        <origin xyz="0 0 0.18" rpy="0 0 0"/>
+        <geometry name="pioneer_geom">
+          <mesh filename="package://p3at_description/meshes/p3at_meshes/chassis.dae"/>
+        </geometry>
+      </visual>
+      <collision>
+        <origin xyz="0 0 0.18" rpy="0 0 0"/>
+        <geometry>
+          <box size="0.501 0.3 0.19"/>
+        </geometry>
+      </collision>
+    </link>
+    <link name="p3at_front_left_wheel">
+      <inertial>
+        <mass value="1.5"/>
+        <origin xyz="0 0 0"/>
+        <inertia ixx="0.005240625" ixy="0" ixz="0"
+          iyy="0.005240625" iyz="0" izz="0.009075"/>
+      </inertial>
+      <visual name="visual">
+        <origin xyz="0 0 0" rpy="0 0 0"/>
+        <geometry name="geom">
+          <mesh filename="package://p3at_description/meshes/p3at_meshes/wheel.dae"/>
+        </geometry>
+      </visual>
+      <collision>
+        <origin xyz="0 0 0" rpy="0 0 0"/>
+        <geometry>
+          <cylinder radius="0.110" length="0.075"/>
+        </geometry>
+      </collision>
+    </link>
+    <joint name="p3at_front_left_wheel_joint" type="continuous">
+      <axis xyz="0 0 -1"/>
+      <limit effort="100" velocity="100" />
+      <joint_properties damping="0.7"/>
+      <origin xyz="0.125 0.2010 0.11" rpy="1.5707 0 0"/>
+      <parent link="base_link"/>
+      <child link="p3at_front_left_wheel"/>
+    </joint>
+    <link name="p3at_front_right_wheel">
+      <inertial>
+        <mass value="1.5"/>
+        <origin xyz="0 0 0"/>
+        <inertia ixx="0.005240625" ixy="0" ixz="0"
+          iyy="0.005240625" iyz="0" izz="0.009075"/>
+      </inertial>
+      <visual name="visual">
+        <origin xyz="0 0 0" rpy="0 0 0"/>
+        <geometry name="geom">
+          <mesh filename="package://p3at_description/meshes/p3at_meshes/wheel.dae"/>
+        </geometry>
+      </visual>
+      <collision>
+        <origin xyz="0 0 0" rpy="0 0 0"/>
+        <geometry>
+          <cylinder radius="0.110" length="0.075"/>
+        </geometry>
+      </collision>
+    </link>
+    <joint name="p3at_front_right_wheel_joint" type="continuous">
+      <axis xyz="0 0 -1"/>
+      <limit effort="100" velocity="100" />
+      <joint_properties damping="0.7"/>
+      <origin xyz="0.125 -0.2010 0.11" rpy="1.5707 0 0"/>
+      <parent link="base_link"/>
+      <child link="p3at_front_right_wheel"/>
+    </joint>
+    <link name="p3at_rear_left_wheel">
+      <inertial>
+        <mass value="1.5"/>
+        <origin xyz="0 0 0"/>
+        <inertia ixx="0.005240625" ixy="0" ixz="0"
+          iyy="0.005240625" iyz="0" izz="0.009075"/>
+      </inertial>
+      <visual name="visual">
+        <origin xyz="0 0 0" rpy="0 0 0"/>
+        <geometry name="geom">
+          <mesh filename="package://p3at_description/meshes/p3at_meshes/wheel.dae"/>
+        </geometry>
+      </visual>
+      <collision>
+        <origin xyz="0 0 0" rpy="0 0 0"/>
+        <geometry>
+          <cylinder radius="0.110" length="0.075"/>
+        </geometry>
+      </collision>
+    </link>
+    <joint name="p3at_rear_left_wheel_joint" type="continuous">
+      <axis xyz="0 0 -1"/>
+      <limit effort="100" velocity="100" />
+      <joint_properties damping="0.7"/>
+      <origin xyz="-0.125 0.2010 0.11" rpy="1.5707 0 0"/>
+      <parent link="base_link"/>
+      <child link="p3at_rear_left_wheel"/>
+    </joint>
+    <link name="p3at_rear_right_wheel">
+      <inertial>
+        <mass value="1.5"/>
+        <origin xyz="0 0 0"/>
+        <inertia ixx="0.005240625" ixy="0" ixz="0"
+          iyy="0.005240625" iyz="0" izz="0.009075"/>
+      </inertial>
+      <visual name="visual">
+        <origin xyz="0 0 0" rpy="0 0 0"/>
+        <geometry name="geom">
+          <mesh filename="package://p3at_description/meshes/p3at_meshes/wheel.dae"/>
+        </geometry>
+      </visual>
+      <collision>
+        <origin xyz="0 0 0" rpy="0 0 0"/>
+        <geometry>
+          <cylinder radius="0.110" length="0.075"/>
+        </geometry>
+      </collision>
+    </link>
+    <joint name="p3at_rear_right_wheel_joint" type="continuous">
+      <axis xyz="0 0 -1"/>
+      <limit effort="100" velocity="100" />
+      <joint_properties damping="0.7"/>
+      <origin xyz="-0.125 -0.2010 0.11" rpy="1.5707 0 0"/>
+      <parent link="base_link"/>
+      <child link="p3at_rear_right_wheel"/>
+    </joint>
+    <gazebo>
+      <plugin name="skid_steer_drive_controller" filename="libgazebo_ros_skid_steer_drive.so">
+        <updateRate>10.0</updateRate>
+        <robotNamespace>/</robotNamespace>
+        <leftFrontJoint>p3at_front_left_wheel_joint</leftFrontJoint>
+        <rightFrontJoint>p3at_front_right_wheel_joint</rightFrontJoint>
+        <leftRearJoint>p3at_rear_left_wheel_joint</leftRearJoint>
+        <rightRearJoint>p3at_rear_right_wheel_joint</rightRearJoint>
+        <wheelSeparation>0.4</wheelSeparation>
+        <wheelDiameter>0.215</wheelDiameter>
+        <robotBaseFrame>base_footprint</robotBaseFrame>
+        <torque>200</torque>
+        <commandTopic>cmd_vel</commandTopic>
+        <odometryTopic>odom</odometryTopic>
+        <odometryFrame>odom</odometryFrame>
+        <broadcastTF>true</broadcastTF>
+        <publishWheelJointState>true</publishWheelJointState>
+      </plugin>
+    </gazebo>
+    <gazebo>
+      <plugin name="p3d" filename="libgazebo_ros_p3d.so">
+        <bodyName>base_footprint</bodyName>
+        <topicName>base_pose_ground_truth</topicName>
+        <frameName>map</frameName>
+        <updateRate>10.0</updateRate>
+      </plugin>
+    </gazebo>
+  </xacro:macro>
 </robot>
